File: pcb/Lucas11-Keychain.kicad_pcb (KiCad board)
At the start: 2 copper layers, 81 x 50 mm, 6 parts

Commit message: as
Other:
- outline, holes or cut-outs redrawn
Changed lines of the file:
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@@
 			(at 0 0 0)
 			(layer "F.SilkS")
+			(hide yes)
 			(effects
 				(font
@@
 	)
 	(gr_circle
-		(center 14.2875 30.95625)
-		(end 14.2875 32.146875)
+		(center 88.10625 38.1)
+		(end 88.10625 39.290625)
 		(stroke
 			(width 0.05)
@@
 	)
 	(gr_text "Hola soy Lucas Altamirano y me encanta los PCBs, Programacion y 3D.\nContactame en altamiranolucas2013@gmail.com .\nVisita lucas11.dev :)"
-		(at 69.05625 19.05 0)
+		(at 90.4875 19.05 0)
 		(layer "B.SilkS")
 		(effects

Commit message: a
Parts:
- added G***: LOGO, LOGO, F.Cu at (38.1, 50.0)
- added G***: LOGO, LOGO, B.Cu at (26.2, 19.1)
Other:
- outline, holes or cut-outs redrawn
- board text added: "Hola soy Lucas Altamirano. Me encanta los PCBs, Programacion y 3D. Contactame en altamiranolucas2013@gmail.com . Visita lucas11.dev :) Tambien visita hackclub.com. Un Non Profit para aldoldecentes."
- board text added: "ola"
- board text removed: "Hola soy Lucas Altamirano y me encanta los PCBs, Programacion y 3D. Contactame en altamiranolucas2013@gmail.com . Visita lucas11.dev :)"
